File: hardware_design/programmer_board/programmer_board.kicad_pcb (KiCad board)
At the start: 2 copper layers, 47.5 x 18.5 mm, 27 parts, among them J1 SM06B-SRSS-TB(LF)(SN), J2 USB4800-03-A_REVA, Q1 SS8050-G, Q2 SS8050-G, U1 AP2112K-3.3TRG1, U2 TPD2S017DBVR, U3 CH340G, Y1 ECS-120-20-3X-EN-TR

Commit message: device settings storage
Implemented basic library to store device settings on eeprom
Other:
- board text added: "ESP flasher."
- board text removed: "ESP32 flasher."
